File: schema/clock.sch (KiCad schematic (older format))
At the start: 24 parts

Commit message: next step
Parts:
- added R12: R, ~, symbol R
- added VD1, VD2: LED, ~, symbol LED
- renumbered R2 to R1, R8 to R10, R9 to R11, R1 to R2, R10 to R3, R11 to R4, R3 to R5, R4 to R6, R5 to R7, R6 to R8, R7 to R9, VT2 to VT1, VT1 to VT2, VT4 to VT3, VT3 to VT4
Connections:
- net GND: now also R12.2
- net VCC: now also VD1.1
- net at DD2.1 (X1): now also BQ1.1; no longer BQ1.2
- net at DD2.2 (X2): no longer BQ1.1
- new net: VD1.2, VD2.1
- new net: R12.1, VD2.2
Changed lines of the file:
@@
 EESchema Schematic File Version 2
 LIBS:power
-LIBS:conn
+LIBS:timer-cache
 LIBS:gost
-LIBS:device
-LIBS:timer-cache
 LIBS:clock-cache
 EELAYER 27 0
@@
 $EndDescr
 $Comp
-L VT_NPN_BCE VT1
+L VT_NPN_BCE VT2
 U 1 1 52F13E6A
 P 3300 4150
-F 0 "VT1" V 3500 4200 60  0000 R CNN
+F 0 "VT2" V 3500 4200 60  0000 R CNN
 F 1 "КТ315" V 3100 4100 60  0000 R CNN
 F 2 "" H 3300 4150 60  0001 C CNN
@@
 $EndComp
 $Comp
-L POWER_GND #01
+L POWER_GND #?
 U 1 1 52F13E15
 P 7800 2000
-F 0 "#01" V 7750 1950 60  0001 C CNN
+F 0 "#?" V 7750 1950 60  0001 C CNN
 F 1 "POWER_GND" V 7850 1950 60  0001 C CNN
 F 2 "" H 7800 2000 60  0001 C CNN
@@
 $EndComp
 $Comp
-L R R1
+L R R2
 U 1 1 52F1EB00
 P 7050 2600
-F 0 "R1" V 7130 2600 50  0000 C CNN
+F 0 "R2" V 7130 2600 50  0000 C CNN
 F 1 "1к" V 7050 2600 50  0000 C CNN
 F 2 "" H 7050 2600 60  0000 C CNN
@@
 $EndComp
 $Comp
-L R R2
+L R R1
 U 1 1 52F4BCDC
 P 7050 2400
-F 0 "R2" V 6950 2400 50  0000 C CNN
+F 0 "R1" V 6950 2400 50  0000 C CNN
 F 1 "1к" V 7050 2400 50  0000 C CNN
 F 2 "" H 7050 2400 60  0000 C CNN
@@
 $EndComp
 $Comp
-L VT_NPN_BCE VT2
+L VT_NPN_BCE VT1
 U 1 1 52F4C8E0
 P 3300 3450
-F 0 "VT2" V 3500 3500 60  0000 R CNN
+F 0 "VT1" V 3500 3500 60  0000 R CNN
 F 1 "КТ315" V 3100 3400 60  0000 R CNN
 F 2 "" H 3300 3450 60  0001 C CNN
@@
 	6800 3600 6800 3400
 $Comp
-L POWER_VCC #~02
+L POWER_VCC #?
 U 1 1 52F4D84D
 P 6900 3600
-F 0 "#~02" V 6700 3350 60  0001 C CNN
+F 0 "#?" V 6700 3350 60  0001 C CNN
 F 1 "POWER_VCC" H 7050 3500 60  0001 C CNN
 F 2 "" H 6900 3600 60  0000 C CNN
@@
 	6900 3600 6800 3600
 $Comp
-L POWER_GND #03
+L POWER_GND #?
 U 1 1 52F4D89D
 P 9150 2450
-F 0 "#03" V 9100 2400 60  0001 C CNN
+F 0 "#?" V 9100 2400 60  0001 C CNN
 F 1 "POWER_GND" V 9200 2400 60  0001 C CNN
 F 2 "" H 9150 2450 60  0001 C CNN
@@
 $EndComp
 $Comp
-L POWER_VCC #~04
+L POWER_VCC #?
 U 1 1 52F4D8A9
 P 9150 2100
-F 0 "#~04" V 8950 1850 60  0001 C CNN
+F 0 "#?" V 8950 1850 60  0001 C CNN
 F 1 "POWER_VCC" H 9300 2000 60  0001 C CNN
 F 2 "" H 9150 2100 60  0000 C CNN
@@
 	5800 3600 5650 3600
 $Comp
-L POWER_GND #05
+L POWER_GND #?
 U 1 1 52FDA0A6
 P 6950 3800
-F 0 "#05" V 6900 3750 60  0001 C CNN
+F 0 "#?" V 6900 3750 60  0001 C CNN
 F 1 "POWER_GND" V 7000 3750 60  0001 C CNN
 F 2 "" H 6950 3800 60  0001 C CNN
@@
 $EndComp
 $Comp
-L CRYSTAL BQ1
-U 1 1 5327F91C
-P 8550 4500
-F 0 "BQ1" H 8850 4700 60  0000 C CNN
-F 1 "CRYSTAL" H 8850 4300 60  0000 C CNN
-F 2 "~" H 8550 4500 60  0000 C CNN
-F 3 "~" H 8550 4500 60  0000 C CNN
-	1    8550 4500
-	-1   0    0    1
-$EndComp
-$Comp
 L SA_1-2_CL SA2
 U 1 1 5327F9B0
@@
 $EndComp
 $Comp
-L VT_NPN_BCE VT3
+L VT_NPN_BCE VT4
 U 1 1 5327FA48
 P 3300 6500
-F 0 "VT3" V 3500 6550 60  0000 R CNN
+F 0 "VT4" V 3500 6550 60  0000 R CNN
 F 1 "КТ315" V 3100 6450 60  0000 R CNN
 F 2 "" H 3300 6500 60  0001 C CNN
@@
 $EndComp
 $Comp
-L VT_NPN_BCE VT4
+L VT_NPN_BCE VT3
 U 1 1 5327FA4E
 P 3300 5850
-F 0 "VT4" V 3500 5900 60  0000 R CNN
+F 0 "VT3" V 3500 5900 60  0000 R CNN
 F 1 "КТ315" V 3100 5800 60  0000 R CNN
 F 2 "" H 3300 5850 60  0001 C CNN
@@
 $EndComp
 $Comp
-L R R3
+L R R5
 U 1 1 5327FACF
 P 5550 2000
-F 0 "R3" V 5475 2000 50  0000 C CNN
+F 0 "R5" V 5475 2000 50  0000 C CNN
 F 1 "68" V 5550 2000 50  0000 C CNN
 F 2 "" H 5550 2000 60  0000 C CNN
@@
 $EndComp
 $Comp
-L R R4
+L R R6
 U 1 1 5327FAF3
 P 5550 2200
-F 0 "R4" V 5475 2200 50  0000 C CNN
+F 0 "R6" V 5475 2200 50  0000 C CNN
 F 1 "68" V 5550 2200 50  0000 C CNN
 F 2 "" H 5550 2200 60  0000 C CNN
@@
 $EndComp
 $Comp
-L R R5
+L R R7
 U 1 1 5327FB2C
 P 5550 2400
-F 0 "R5" V 5475 2400 50  0000 C CNN
+F 0 "R7" V 5475 2400 50  0000 C CNN
 F 1 "68" V 5550 2400 50  0000 C CNN
 F 2 "" H 5550 2400 60  0000 C CNN
@@
 $EndComp
 $Comp
-L R R6
+L R R8
 U 1 1 5327FB32
 P 5550 2600
-F 0 "R6" V 5475 2600 50  0000 C CNN
+F 0 "R8" V 5475 2600 50  0000 C CNN
 F 1 "68" V 5550 2600 50  0000 C CNN
 F 2 "" H 5550 2600 60  0000 C CNN
@@
 $EndComp
 $Comp
-L R R7
+L R R9
 U 1 1 5327FB38
 P 5550 2800
-F 0 "R7" V 5475 2800 50  0000 C CNN
+F 0 "R9" V 5475 2800 50  0000 C CNN
 F 1 "68" V 5550 2800 50  0000 C CNN
 F 2 "" H 5550 2800 60  0000 C CNN
@@
 $EndComp
 $Comp
-L R R8
+L R R10
 U 1 1 5327FB3E
 P 5550 3000
-F 0 "R8" V 5475 3000 50  0000 C CNN
+F 0 "R10" V 5475 3000 50  0000 C CNN
 F 1 "68" V 5550 3000 50  0000 C CNN
 F 2 "" H 5550 3000 60  0000 C CNN
@@
 $EndComp
 $Comp
-L R R9
+L R R11
 U 1 1 5327FB44
 P 5550 3200
-F 0 "R9" V 5475 3200 50  0000 C CNN
+F 0 "R11" V 5475 3200 50  0000 C CNN
 F 1 "68" V 5550 3200 50  0000 C CNN
 F 2 "" H 5550 3200 60  0000 C CNN
@@
 NoConn ~ 6800 3200
 $Comp
-L R R10
+L R R3
 U 1 1 5327FDFB
 P 7050 2800
-F 0 "R10" V 6950 2800 50  0000 C CNN
+F 0 "R3" V 6950 2800 50  0000 C CNN
 F 1 "1к" V 7050 2800 50  0000 C CNN
 F 2 "" H 7050 2800 60  0000 C CNN
@@
 $EndComp
 $Comp
-L R R11
+L R R4
 U 1 1 5327FE01
 P 7050 3000
-F 0 "R11" V 6950 3000 50  0000 C CNN
+F 0 "R4" V 6950 3000 50  0000 C CNN
 F 1 "1к" V 7050 3000 50  0000 C CNN
 F 2 "" H 7050 3000 60  0000 C CNN
@@
 Connection ~ 7550 2000
 $Comp
-L POWER_VCC #~06
+L POWER_VCC #?
 U 1 1 5327FFC0
 P 6450 4650
-F 0 "#~06" V 6250 4400 60  0001 C CNN
+F 0 "#?" V 6250 4400 60  0001 C CNN
 F 1 "POWER_VCC" H 6600 4550 60  0001 C CNN
 F 2 "" H 6450 4650 60  0000 C CNN
@@
 $EndComp
 $Comp
-L POWER_GND #07
+L POWER_GND #?
 U 1 1 5327FFB1
 P 7450 5250
-F 0 "#07" V 7400 5200 60  0001 C CNN
+F 0 "#?" V 7400 5200 60  0001 C CNN
 F 1 "POWER_GND" V 7500 5200 60  0001 C CNN
 F 2 "" H 7450 5250 60  0001 C CNN
@@
 	3050 3250 3050 6400
 $Comp
-L POWER_VCC #~08
+L POWER_VCC #?
 U 1 1 53280317
 P 3050 3250
-F 0 "#~08" V 2850 3000 60  0001 C CNN
+F 0 "#?" V 2850 3000 60  0001 C CNN
 F 1 "POWER_VCC" H 3200 3150 60  0001 C CNN
 F 2 "" H 3050 3250 60  0000 C CNN
@@
 	5800 5050 6450 5050
 Wire Wire Line
-	7450 4850 8550 4850
-Wire Wire Line
-	8550 4850 8550 4500
+	7450 4850 8300 4850
+Wire Wire Line
+	8300 4850 8300 4500
 Wire Wire Line
 	7450 4650 7950 4650
@@
 	3850 1700 3850 5450
 $Comp
-L PWR_FLAG #FLG09
+L PWR_FLAG #FLG?
 U 1 1 53280E20
 P 8950 2150
-F 0 "#FLG09" H 8950 2245 30  0001 C CNN
+F 0 "#FLG?" H 8950 2245 30  0001 C CNN
 F 1 "PWR_FLAG" H 8950 2330 30  0000 C CNN
 F 2 "" H 8950 2150 60  0000 C CNN
@@
 	8950 2200 8950 2150
 $Comp
-L PWR_FLAG #FLG010
+L PWR_FLAG #FLG?
 U 1 1 53280E6B
 P 8150 5500
-F 0 "#FLG010" H 8150 5595 30  0001 C CNN
+F 0 "#FLG?" H 8150 5595 30  0001 C CNN
 F 1 "PWR_FLAG" H 8150 5680 30  0000 C CNN
 F 2 "" H 8150 5500 60  0000 C CNN
@@
 Connection ~ 6950 3800
 $Comp
-L PWR_FLAG #FLG011
+L PWR_FLAG #FLG?
 U 1 1 532818D0
 P 7400 3800
-F 0 "#FLG011" H 7400 3895 30  0001 C CNN
+F 0 "#FLG?" H 7400 3895 30  0001 C CNN
 F 1 "PWR_FLAG" H 7400 3980 30  0000 C CNN
 F 2 "" H 7400 3800 60  0000 C CNN
@@
 	1    0    0    -1
 $EndComp
+$Comp
+L CRYSTAL BQ1
+U 1 1 53281BA9
+P 7950 4500
+F 0 "BQ1" H 8150 4700 60  0000 C CNN
+F 1 "CRYSTAL" H 8250 4300 60  0001 C CNN
+F 2 "~" H 7950 4500 60  0000 C CNN
+F 3 "~" H 7950 4500 60  0000 C CNN
+	1    7950 4500
+	1    0    0    -1
+$EndComp
+$Comp
+L LED VD1
+U 1 1 53282BF6
+P 9150 4200
+F 0 "VD1" H 9150 4400 60  0000 C CNN
+F 1 "LED" H 9200 4000 60  0000 C CNN
+F 2 "~" H 9150 4200 60  0000 C CNN
+F 3 "~" H 9150 4200 60  0000 C CNN
+	1    9150 4200
+	0    1    1    0
+$EndComp
+$Comp
+L LED VD2
+U 1 1 53282C12
+P 9150 4700
+F 0 "VD2" H 9150 4900 60  0000 C CNN
+F 1 "LED" H 9200 4500 60  0000 C CNN
+F 2 "~" H 9150 4700 60  0000 C CNN
+F 3 "~" H 9150 4700 60  0000 C CNN
+	1    9150 4700
+	0    1    1    0
+$EndComp
+$Comp
+L R R12
+U 1 1 53282C1A
+P 9150 5200
+F 0 "R12" V 9230 5200 50  0000 C CNN
+F 1 "R" V 9150 5200 50  0000 C CNN
+F 2 "~" H 9150 5200 60  0000 C CNN
+F 3 "~" H 9150 5200 60  0000 C CNN
+	1    9150 5200
+	1    0    0    -1
+$EndComp
+$Comp
+L POWER_GND #?
+U 1 1 53282C27
+P 9150 5450
+F 0 "#?" V 9100 5400 60  0001 C CNN
+F 1 "POWER_GND" V 9200 5400 60  0001 C CNN
+F 2 "" H 9150 5450 60  0001 C CNN
+F 3 "" H 9150 5450 60  0001 C CNN
+	1    9150 5450
+	1    0    0    -1
+$EndComp
+$Comp
+L POWER_VCC #?
+U 1 1 53282C2D
+P 9150 3950
+F 0 "#?" V 8950 3700 60  0001 C CNN
+F 1 "POWER_VCC" H 9300 3850 60  0001 C CNN
+F 2 "" H 9150 3950 60  0000 C CNN
+F 3 "" H 9150 3950 60  0000 C CNN
+	1    9150 3950
+	0    1    -1   0
+$EndComp
 $EndSCHEMATC

Commit message: next step
Parts:
- added R13, R14: R, ~, symbol R
Connections:
- net VCC: now also R13.1
- net at DD1.4 (PA1), DD2.6 (SCL): now also R14.2
- net at DD1.5 (PA0), DD2.5 (SDA): now also R13.2
Changed lines of the file:
@@
 EESchema Schematic File Version 2
 LIBS:power
-LIBS:timer-cache
 LIBS:gost
 LIBS:clock-cache
@@
 Sheet 1 1
 Title ""
-Date "18 mar 2014"
+Date "19 mar 2014"
 Rev ""
 Comp ""
@@
 L POWER_VCC #?
 U 1 1 5327FFC0
-P 6450 4650
-F 0 "#?" V 6250 4400 60  0001 C CNN
-F 1 "POWER_VCC" H 6600 4550 60  0001 C CNN
-F 2 "" H 6450 4650 60  0000 C CNN
-F 3 "" H 6450 4650 60  0000 C CNN
-	1    6450 4650
+P 6450 4450
+F 0 "#?" V 6250 4200 60  0001 C CNN
+F 1 "POWER_VCC" H 6600 4350 60  0001 C CNN
+F 2 "" H 6450 4450 60  0000 C CNN
+F 3 "" H 6450 4450 60  0000 C CNN
+	1    6450 4450
 	0    1    -1   0
 $EndComp
@@
 	0    1    -1   0
 $EndComp
+$Comp
+L R R14
+U 1 1 53296CF2
+P 6250 4700
+F 0 "R14" H 6350 4700 50  0000 C CNN
+F 1 "R" V 6250 4700 50  0000 C CNN
+F 2 "~" H 6250 4700 60  0000 C CNN
+F 3 "~" H 6250 4700 60  0000 C CNN
+	1    6250 4700
+	1    0    0    -1
+$EndComp
+$Comp
+L R R13
+U 1 1 53296CF8
+P 6050 4700
+F 0 "R13" H 5950 4750 50  0000 C CNN
+F 1 "R" V 6050 4700 50  0000 C CNN
+F 2 "~" H 6050 4700 60  0000 C CNN
+F 3 "~" H 6050 4700 60  0000 C CNN
+	1    6050 4700
+	1    0    0    -1
+$EndComp
+Wire Wire Line
+	6450 4450 6050 4450
+Wire Wire Line
+	6450 4650 6450 4450
+Wire Wire Line
+	6250 4950 6250 5050
+Connection ~ 6250 5050
+Wire Wire Line
+	6050 4950 6050 5250
+Connection ~ 6050 5250
 $EndSCHEMATC

Commit message: edit
Parts:
- added C1: 1u, ~, symbol CAPP
Connections:
- net GND: now also C1.1
- net VCC: now also C1.2
Changed lines of the file:
@@
 EESchema Schematic File Version 2
 LIBS:power
+LIBS:timer-cache
 LIBS:gost
 LIBS:clock-cache
@@
 Sheet 1 1
 Title ""
-Date "19 mar 2014"
+Date "22 mar 2014"
 Rev ""
 Comp ""
@@
 L POWER_GND #?
 U 1 1 52F4D89D
-P 9150 2450
-F 0 "#?" V 9100 2400 60  0001 C CNN
-F 1 "POWER_GND" V 9200 2400 60  0001 C CNN
-F 2 "" H 9150 2450 60  0001 C CNN
-F 3 "" H 9150 2450 60  0001 C CNN
-	1    9150 2450
+P 9150 2600
+F 0 "#?" V 9100 2550 60  0001 C CNN
+F 1 "POWER_GND" V 9200 2550 60  0001 C CNN
+F 2 "" H 9150 2600 60  0001 C CNN
+F 3 "" H 9150 2600 60  0001 C CNN
+	1    9150 2600
 	1    0    0    -1
 $EndComp
@@
 L POWER_VCC #?
 U 1 1 52F4D8A9
-P 9150 2100
-F 0 "#?" V 8950 1850 60  0001 C CNN
-F 1 "POWER_VCC" H 9300 2000 60  0001 C CNN
-F 2 "" H 9150 2100 60  0000 C CNN
-F 3 "" H 9150 2100 60  0000 C CNN
-	1    9150 2100
+P 9150 1850
+F 0 "#?" V 8950 1600 60  0001 C CNN
+F 1 "POWER_VCC" H 9300 1750 60  0001 C CNN
+F 2 "" H 9150 1850 60  0000 C CNN
+F 3 "" H 9150 1850 60  0000 C CNN
+	1    9150 1850
 	0    -1   -1   0
 $EndComp
@@
 $EndComp
 Wire Wire Line
-	9150 2200 9150 2100
-Wire Wire Line
-	9150 2300 9150 2450
+	9150 2200 9150 1850
+Wire Wire Line
+	9150 2300 9150 2600
 Wire Wire Line
 	7200 2000 7800 2000
@@
 VT1
 Wire Wire Line
-	6450 5250 5650 5250
-Wire Wire Line
-	5650 5250 5650 3600
+	5650 5250 6450 5250
+Wire Wire Line
+	5650 3600 5650 5250
 Wire Wire Line
 	5800 3800 5800 5050
@@
 L PWR_FLAG #FLG?
 U 1 1 53280E20
-P 8950 2150
-F 0 "#FLG?" H 8950 2245 30  0001 C CNN
-F 1 "PWR_FLAG" H 8950 2330 30  0000 C CNN
-F 2 "" H 8950 2150 60  0000 C CNN
-F 3 "" H 8950 2150 60  0000 C CNN
-	1    8950 2150
+P 8950 1900
+F 0 "#FLG?" H 8950 1995 30  0001 C CNN
+F 1 "PWR_FLAG" H 8950 2080 30  0000 C CNN
+F 2 "" H 8950 1900 60  0000 C CNN
+F 3 "" H 8950 1900 60  0000 C CNN
+	1    8950 1900
 	1    0    0    -1
 $EndComp
@@
 	9150 2200 8950 2200
 Wire Wire Line
-	8950 2200 8950 2150
+	8950 2200 8950 1900
 $Comp
 L PWR_FLAG #FLG?
@@
 	6050 4950 6050 5250
 Connection ~ 6050 5250
+$Comp
+L CAPP C1
+U 1 1 532DF229
+P 8550 2000
+F 0 "C1" H 8650 1900 60  0000 C CNN
+F 1 "1u" H 8700 1650 60  0000 C CNN
+F 2 "~" H 8550 2000 60  0000 C CNN
+F 3 "~" H 8550 2000 60  0000 C CNN
+	1    8550 2000
+	1    0    0    -1
+$EndComp
+Wire Wire Line
+	8550 2000 8950 2000
+Connection ~ 8950 2000
+Wire Wire Line
+	8550 2450 9150 2450
+Connection ~ 9150 2450
 $EndSCHEMATC
